File: new/clock_esp32_pcb.kicad_sch (KiCad schematic)
At the start: 10 parts

Commit message: final routing completed
Parts:
- BUZZER1, pwr_IN1: footprint Connector_PinSocket_1.27mm:PinSocket_1x02_P1.27mm_Vertical -> Connector_PinSocket_2.54mm:PinSocket_1x02_P2.54mm_Vertical
- C1: footprint (none) -> Capacitor_THT:C_Radial_D6.3mm_H5.0mm_P2.50mm
- ESP_left1, ESP_right1: footprint Connector_PinSocket_1.27mm:PinSocket_1x19_P1.27mm_Vertical -> Connector_PinSocket_2.54mm:PinSocket_1x19_P2.54mm_Vertical
- RTC1: footprint Connector_PinSocket_1.27mm:PinSocket_1x06_P1.27mm_Vertical -> Connector_PinSocket_2.54mm:PinSocket_1x06_P2.54mm_Vertical
- lcd_I2C1: footprint Connector_PinSocket_1.27mm:PinSocket_1x04_P1.27mm_Vertical -> Connector_PinSocket_2.54mm:PinSocket_1x04_P2.54mm_Vertical
Changed lines of the file:
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@@
 			)
 		)
-		(property "Footprint" "Connector_PinSocket_1.27mm:PinSocket_1x06_P1.27mm_Vertical"
+		(property "Footprint" "Connector_PinSocket_2.54mm:PinSocket_1x06_P2.54mm_Vertical"
 			(at 236.22 67.31 0)
 			(effects
@@
 			)
 		)
-		(property "Footprint" ""
+		(property "Footprint" "Capacitor_THT:C_Radial_D6.3mm_H5.0mm_P2.50mm"
 			(at 93.6752 138.43 0)
 			(effects
@@
 			)
 		)
-		(property "Footprint" "Connector_PinSocket_1.27mm:PinSocket_1x02_P1.27mm_Vertical"
+		(property "Footprint" "Connector_PinSocket_2.54mm:PinSocket_1x02_P2.54mm_Vertical"
 			(at 207.01 132.08 0)
 			(effects
@@
 			)
 		)
-		(property "Footprint" "Connector_PinSocket_1.27mm:PinSocket_1x02_P1.27mm_Vertical"
+		(property "Footprint" "Connector_PinSocket_2.54mm:PinSocket_1x02_P2.54mm_Vertical"
 			(at 118.11 128.27 0)
 			(effects
@@
 			)
 		)
-		(property "Footprint" "Connector_PinSocket_1.27mm:PinSocket_1x04_P1.27mm_Vertical"
+		(property "Footprint" "Connector_PinSocket_2.54mm:PinSocket_1x04_P2.54mm_Vertical"
 			(at 234.95 105.41 0)
 			(effects
@@
 			)
 		)
-		(property "Footprint" "Connector_PinSocket_1.27mm:PinSocket_1x19_P1.27mm_Vertical"
+		(property "Footprint" "Connector_PinSocket_2.54mm:PinSocket_1x19_P2.54mm_Vertical"
 			(at 157.48 101.6 0)
 			(effects
@@
 			)
 		)
-		(property "Footprint" "Connector_PinSocket_1.27mm:PinSocket_1x19_P1.27mm_Vertical"
+		(property "Footprint" "Connector_PinSocket_2.54mm:PinSocket_1x19_P2.54mm_Vertical"
 			(at 147.32 101.6 0)
 			(effects
